File: SRP3075_PowerSupply/KiCad/SRP3075_PowerSupply.kicad_sch (KiCad schematic)
At the start: 20 parts, among them J1 To Main Board, K1 Hamlin 701-12-5, M1 Motor_AC_DV, M2 Fan, SW1 Control Panel - Power Switch, T1 DSI-8382-2, U2 UA7912

Commit message: Updated resistor value
Parts:
- RX1: value 620 -> 1.2k
Changed lines of the file:
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@@
 			)
 		)
-		(property "Value" "620"
+		(property "Value" "1.2k"
 			(at 110.49 166.3699 0)
 			(effects
